Commit message: ros2_control issues

File: description/gazebo_control.xacro (robot description, xacro)
@@ -6,5 +6,5 @@
             <left_joint>left_wheel_joint</left_joint>
             <right_joint>right_wheel_joint</right_joint>
-            <wheel_separation>0.575</wheel_separation>
+            <wheel_separation>0.58</wheel_separation>
             <wheel_diameter>0.12</wheel_diameter>
             <!-- Limits -->

File: description/lidar.xacro (robot description, xacro)
@@ -22,5 +22,5 @@
         <parent link="chassis_link"/>
         <child link="laser_frame"/>
-        <origin xyz="0.195 0 0.1025" rpy="0 0 0"/>
+        <origin xyz="0.19 0 0.1025" rpy="0 0 0"/>
     </joint>
     <gazebo reference="laser_frame">
@@ -28,5 +28,5 @@
         <sensor name="laser" type="ray">
             <pose> 0 0 0 0 0 0 </pose>
-            <visualize>true</visualize>
+            <visualize>false</visualize>
             <update_rate>10</update_rate>
             <ray>

File: description/robot.urdf.xacro (robot description, xacro)
@@ -1,7 +1,12 @@
 <?xml version="1.0"?>
 <robot xmlns:xacro="http://www.ros.org/wiki/xacro"  name="robot">
+    <xacro:arg name="use_ros2_control" default="true"/>
     <xacro:include filename="robot_core.xacro" />
-    <!-- <xacro:include filename="gazebo_control.xacro" /> -->
-    <xacro:include filename="ros2_control.xacro" />
+    <xacro:if value="$(arg use_ros2_control)">
+        <xacro:include filename="ros2_control.xacro" />
+    </xacro:if>
+    <xacro:unless value="$(arg use_ros2_control)">
+        <xacro:include filename="gazebo_control.xacro" />
+    </xacro:unless>
     <xacro:include filename="lidar.xacro" />
 </robot>

File: description/robot_core.xacro (robot description, xacro)
@@ -2,4 +2,18 @@
 <robot xmlns:xacro="http://www.ros.org/wiki/xacro" >
     <xacro:include filename="inertial_macros.xacro"/>
+    <xacro:property name="chassis_length" value="0.49"/>
+    <xacro:property name="chassis_width" value="0.49"/>
+    <xacro:property name="chassis_height" value="0.15"/>
+    <xacro:property name="chassis_mass" value="5.0"/>
+    <xacro:property name="wheel_radius" value="0.06"/>
+    <xacro:property name="wheel_thickness" value="0.06"/>
+    <xacro:property name="wheel_mass" value="0.2"/>
+    <xacro:property name="wheel_offset_x" value="0.226"/>
+    <xacro:property name="wheel_offset_y" value="0.1485"/>
+    <xacro:property name="wheel_offset_z" value="0.01"/>
+    <xacro:property name="caster_wheel_radius" value="0.01"/>
+    <xacro:property name="caster_wheel_mass" value="0.01"/>
+    <xacro:property name="caster_wheel_offset_x" value="0.075"/>
+    <xacro:property name="caster_wheel_offset_z" value="${wheel_offset_z - wheel_radius + caster_wheel_radius}"/>
     <material name="blue">
       <color rgba="0 0 0.8 1"/>
@@ -21,5 +35,5 @@
         <visual>
             <geometry>
-                <box size="0.5 0.5 0.15"/>
+                <box size="0.49 0.49 0.15"/>
             </geometry>
             <material name="white"/>
@@ -28,9 +42,9 @@
         <collision>
             <geometry>
-                <box size="0.5 0.5 0.15"/>
+                <box size="0.49 0.49 0.15"/>
             </geometry>
             <origin xyz="0.0 0.0 0.0" rpy="0.0 0.0 0.0"/>
         </collision>
-        <xacro:inertial_box mass="5" x="0.5" y="0.5" z="0.15">
+        <xacro:inertial_box mass="5" x="0.49" y="0.49" z="0.15">
             <origin xyz="0 0 0" rpy="0 0 0"/>
         </xacro:inertial_box>
@@ -49,5 +63,5 @@
         <visual>
             <geometry>
-                <cylinder radius="0.06" length="0.075"/>
+                <cylinder radius="0.06" length="0.06"/>
             </geometry>
             <material name="black"/>
@@ -56,14 +70,14 @@
         <collision>
             <geometry>
-            <cylinder radius="0.06" length="0.075"/>
+                <sphere radius="0.06"/>
             </geometry>
             <origin rpy="1.5708 0 0" xyz="0 0 0"/>
         </collision>
-        <xacro:inertial_cylinder mass="0.2" length="0.075" radius="0.06">
+        <xacro:inertial_cylinder mass="0.2" length="0.06" radius="0.06">
             <origin xyz="0 0 0" rpy="0 0 0"/>
         </xacro:inertial_cylinder>
     </link>
     <joint name="right_wheel_joint" type="continuous">
-        <origin xyz="0.13 0.2875 -0.09" rpy="0 0 0" />
+        <origin xyz="0.125 0.29 -0.09" rpy="0 0 0" />
         <parent link="base_link" />
         <child link="right_wheel" />
@@ -77,5 +91,5 @@
         <visual>
             <geometry>
-                <cylinder radius="0.06" length="0.075"/>
+                <cylinder radius="0.06" length="0.06"/>
             </geometry>
             <material name="black"/>
@@ -85,13 +99,13 @@
             <origin rpy="1.5708 0 0" xyz="0 0 0"/>
             <geometry>
-                <cylinder radius="0.06" length="0.075"/>
+                <sphere radius="0.06"/>
             </geometry>
         </collision>
-        <xacro:inertial_cylinder mass="0.2" length="0.075" radius="0.06">
+        <xacro:inertial_cylinder mass="0.2" length="0.06" radius="0.06">
             <origin xyz="0 0 0" rpy="0 0 0"/>
         </xacro:inertial_cylinder>
     </link>
     <joint name="left_wheel_joint" type="continuous">
-        <origin xyz="0.13 -0.2875 -0.09" rpy="0 0 0" />
+        <origin xyz="0.125 -0.29 -0.09" rpy="0 0 0" />
         <parent link="base_link" />
         <child link="left_wheel" />
@@ -121,5 +135,5 @@
     </link>
     <joint name="caster_wheel_joint" type="fixed">
-        <origin xyz="-0.25 0 -0.110" rpy="0 0 0" />
+        <origin xyz="-0.24 0 -0.110" rpy="0 0 0" />
         <parent link="chassis_link" />
         <child link="caster_wheel" />
