Commit message: Arreglando orientacion

File: description/lidar.xacro (robot description, xacro)
@@ -22,5 +22,5 @@
         <parent link="chassis_link"/>
         <child link="laser_frame"/>
-        <origin xyz="0.19 0 0.1025" rpy="0 0 0"/>
+        <origin xyz="-0.19 0 0.1025" rpy="0 0 0"/>
     </joint>
     <gazebo reference="laser_frame">

File: description/robot_core.xacro (robot description, xacro)
@@ -79,5 +79,5 @@
     </link>
     <joint name="right_wheel_joint" type="continuous">
-        <origin xyz="0.125 -0.29 -0.09" rpy="0 0 0" />
+        <origin xyz="-0.125 0.29 -0.09" rpy="0 0 0" />
         <parent link="base_link" />
         <child link="right_wheel" />
@@ -107,5 +107,5 @@
     </link>
     <joint name="left_wheel_joint" type="continuous">
-        <origin xyz="0.125 0.29 -0.09" rpy="0 0 0" />
+        <origin xyz="-0.125 -0.29 -0.09" rpy="0 0 0" />
         <parent link="base_link" />
         <child link="left_wheel" />
@@ -135,5 +135,5 @@
     </link>
     <joint name="caster_wheel_joint" type="fixed">
-        <origin xyz="-0.24 0 -0.110" rpy="0 0 0" />
+        <origin xyz="0.24 0 -0.110" rpy="0 0 0" />
         <parent link="chassis_link" />
         <child link="caster_wheel" />

Commit message: Fixing odometry

File: description/lidar.xacro (robot description, xacro)
@@ -22,5 +22,5 @@
         <parent link="chassis_link"/>
         <child link="laser_frame"/>
-        <origin xyz="-0.19 0 0.1025" rpy="0 0 0"/>
+        <origin xyz="0.19 0 0.1025" rpy="0 0 3.1415"/>
     </joint>
     <gazebo reference="laser_frame">

File: description/robot_core.xacro (robot description, xacro)
@@ -66,5 +66,5 @@
             </geometry>
             <material name="black"/>
-            <origin rpy="1.5708 0 0" xyz="0 0 0"/>
+            <origin rpy="0 0 0" xyz="0 0 0"/>
         </visual>
         <collision>
@@ -72,5 +72,5 @@
                 <sphere radius="0.06"/>
             </geometry>
-            <origin rpy="1.5708 0 0" xyz="0 0 0"/>
+            <origin rpy="0 0 0" xyz="0 0 0"/>
         </collision>
         <xacro:inertial_cylinder mass="0.2" length="0.06" radius="0.06">
@@ -79,8 +79,8 @@
     </link>
     <joint name="right_wheel_joint" type="continuous">
-        <origin xyz="-0.125 0.29 -0.09" rpy="0 0 0" />
+        <origin xyz="0.125 -0.29 -0.09" rpy="-1.5708 0 0" />
         <parent link="base_link" />
         <child link="right_wheel" />
-        <axis xyz="0 1 0" />
+        <axis xyz="0 0 1" />
     </joint>
     <gazebo reference="right_wheel">
@@ -94,8 +94,8 @@
             </geometry>
             <material name="black"/>
-            <origin rpy="1.5708 0 0" xyz="0 0 0"/>
+            <origin rpy="0 0 0" xyz="0 0 0"/>
         </visual>
         <collision>
-            <origin rpy="1.5708 0 0" xyz="0 0 0"/>
+            <origin rpy="0 0 0" xyz="0 0 0"/>
             <geometry>
                 <sphere radius="0.06"/>
@@ -107,8 +107,8 @@
     </link>
     <joint name="left_wheel_joint" type="continuous">
-        <origin xyz="-0.125 -0.29 -0.09" rpy="0 0 0" />
+        <origin xyz="0.125 0.29 -0.09" rpy="-1.5708 0 0" />
         <parent link="base_link" />
         <child link="left_wheel" />
-        <axis xyz="0 1 0" />
+        <axis xyz="0 0 1" />
     </joint>
     <gazebo reference="left_wheel">
@@ -135,5 +135,5 @@
     </link>
     <joint name="caster_wheel_joint" type="fixed">
-        <origin xyz="0.24 0 -0.110" rpy="0 0 0" />
+        <origin xyz="-0.24 0 -0.110" rpy="0 0 0" />
         <parent link="chassis_link" />
         <child link="caster_wheel" />

File: description/ros2_control.xacro (robot description, xacro)
@@ -11,5 +11,5 @@
                 <param name="baud_rate">57600</param>
                 <param name="timeout">1000</param>
-                <param name="enc_counts_per_rev">8384</param>
+                <param name="enc_counts_per_rev">6533</param>
             </hardware>
             <joint name="left_wheel_joint">

Commit message: addingfiles

File: description/lidar.xacro (robot description, xacro)
@@ -34,6 +34,6 @@
                     <horizontal>
                         <samples>360</samples>
-                        <min_angle>-3.14159</min_angle>
-                        <max_angle>3.14159</max_angle>
+                        <min_angle>-2.356</min_angle>
+                        <max_angle>2.356</max_angle>
                     </horizontal>
                 </scan>

File: description/robot_core.xacro (robot description, xacro)
@@ -30,4 +30,12 @@
     <!-- BASE LINK -->
     <link name="base_link">
+    </link>
+    <!-- BASE_FOOTPRINT LINK -->
+    <joint name="base_footprint_joint" type="fixed">
+        <parent link="base_link"/>
+        <child link="base_footprint"/>
+        <origin xyz="0 0 0" rpy="0 0 0"/>
+    </joint>
+    <link name="base_footprint">
     </link>
     <!--CHASSIS OF THE ROBOT-->
@@ -79,5 +87,5 @@
     </link>
     <joint name="right_wheel_joint" type="continuous">
-        <origin xyz="0.125 -0.29 -0.09" rpy="-1.5708 0 0" />
+        <origin xyz="0.125 -0.295 -0.09" rpy="-1.5708 0 0" />
         <parent link="base_link" />
         <child link="right_wheel" />
@@ -107,5 +115,5 @@
     </link>
     <joint name="left_wheel_joint" type="continuous">
-        <origin xyz="0.125 0.29 -0.09" rpy="-1.5708 0 0" />
+        <origin xyz="0.125 0.295 -0.09" rpy="-1.5708 0 0" />
         <parent link="base_link" />
         <child link="left_wheel" />

Commit message: adding humble

File: description/lidar.xacro (robot description, xacro)
@@ -34,6 +34,6 @@
                     <horizontal>
                         <samples>360</samples>
-                        <min_angle>-2.356</min_angle>
-                        <max_angle>2.356</max_angle>
+                        <min_angle>-3.14</min_angle>
+                        <max_angle>3.14</max_angle>
                     </horizontal>
                 </scan>

File: description/robot_core.xacro (robot description, xacro)
@@ -87,5 +87,5 @@
     </link>
     <joint name="right_wheel_joint" type="continuous">
-        <origin xyz="0.125 -0.295 -0.09" rpy="-1.5708 0 0" />
+        <origin xyz="0 -0.29 -0.09" rpy="-1.5708 0 0" />
         <parent link="base_link" />
         <child link="right_wheel" />
@@ -115,5 +115,5 @@
     </link>
     <joint name="left_wheel_joint" type="continuous">
-        <origin xyz="0.125 0.295 -0.09" rpy="-1.5708 0 0" />
+        <origin xyz="0 0.29 -0.09" rpy="-1.5708 0 0" />
         <parent link="base_link" />
         <child link="left_wheel" />
@@ -153,4 +153,34 @@
         <mu2 value="0.001"/>
     </gazebo>
+    <!--CASTER_WHEEL2-->
+    <link name="caster_wheel2">
+        <visual>
+            <geometry>
+                <sphere radius="0.035"/>
+            </geometry>
+            <material name="green"/>
+            <origin rpy="0 0 0" xyz="0 0 0"/>
+        </visual>
+        <collision>
+            <origin rpy="0 0 0" xyz="0 0 0"/>
+            <geometry>
+                <sphere radius="0.035"/>
+            </geometry>
+        </collision>
+        <xacro:inertial_sphere mass="0.1" radius="0.035">
+            <origin xyz="0 0 0" rpy="0 0 0"/>
+        </xacro:inertial_sphere>
+    </link>
+    <joint name="caster_wheel_joint2" type="fixed">
+        <origin xyz="0.24 0 -0.110" rpy="0 0 0" />
+        <parent link="chassis_link" />
+        <child link="caster_wheel2" />
+        <axis xyz="0 0 0" />
+    </joint>
+    <gazebo reference="caster_wheel2">
+        <material>Gazebo/Green</material>
+        <mu1 value="0.001"/>
+        <mu2 value="0.001"/>
+    </gazebo>
     <!--LIGHT TUBE-->
     <link name="light_tube">

File: description/ros2_control.xacro (robot description, xacro)
@@ -15,6 +15,6 @@
             <joint name="left_wheel_joint">
                 <command_interface name="velocity">
-                    <param name="min">-10</param>
-                    <param name="max">10</param>
+                    <param name="min">-0.2</param>
+                    <param name="max">0.2</param>
                 </command_interface>
                 <state_interface name="velocity"/>
@@ -23,6 +23,6 @@
             <joint name="right_wheel_joint">
                 <command_interface name="velocity">
-                    <param name="min">-10</param>
-                    <param name="max">10</param>
+                    <param name="min">-0.2</param>
+                    <param name="max">0.2</param>
                 </command_interface>
                 <state_interface name="velocity"/>

Commit message: Modified

File: description/lidar.xacro (robot description, xacro)
@@ -2,4 +2,9 @@
 <robot xmlns:xacro="http://www.ros.org/wiki/xacro">
     <!--RPLIDAR-->
+    <joint name="laser_joint" type="fixed">
+        <parent link="chassis_link"/>
+        <child link="laser_frame"/>
+        <origin xyz="0.19 0 0.1025" rpy="0 0 3.1415"/>
+    </joint>
     <link name="laser_frame">
         <visual>
@@ -7,5 +12,5 @@
                 <cylinder radius="0.035" length="0.055"/>
             </geometry>
-            <material name="red"/>
+            <material name="white"/>
             <origin xyz="0 0 0"/>
         </visual>
@@ -19,11 +24,6 @@
         </xacro:inertial_cylinder>
     </link>
-    <joint name="laser_joint" type="fixed">
-        <parent link="chassis_link"/>
-        <child link="laser_frame"/>
-        <origin xyz="0.19 0 0.1025" rpy="0 0 3.1415"/>
-    </joint>
     <gazebo reference="laser_frame">
-        <material>Gazebo/Red</material>
+        <material>Gazebo/White</material>
         <sensor name="laser" type="ray">
             <pose> 0 0 0 0 0 0 </pose>
